File: 3340_VCO/Kicad Project/3340_VCO.kicad_sch (KiCad schematic)
At the start: 74 parts, among them J1 FM_IN, J10 Conn_1A, J11 Conn_1B, J12 Conn_2B, J13 Conn_2A, J2 PWM_IN, J3 PULSE_OUT, J4 SYNC_IN, J5 SAW_OUT, J6 V/OCT_IN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

Commit message: Recent updates for eurorack pcbs
Parts:
- removed J11: Conn_1B, Connector_PinHeader_2.54mm:PinHeader_1x07_P2.54mm_Vertical, symbol Connector:Conn_01x07_Socket
- removed J12: Conn_2B, Connector_PinHeader_2.54mm:PinHeader_1x07_P2.54mm_Vertical, symbol Connector:Conn_01x07_Socket
- added J11: Conn_1A, Connector_PinSocket_2.54mm:PinSocket_1x07_P2.54mm_Vertical, symbol Connector:Conn_01x07_Pin
- added J12: Conn_2A, Connector_PinSocket_2.54mm:PinSocket_1x07_P2.54mm_Vertical, symbol Connector:Conn_01x07_Pin
- J10: value Conn_1A -> Conn_1B
- J13: value Conn_2A -> Conn_2B
- U1: footprint Package_DIP:DIP-16_W10.16mm_LongPads -> Package_DIP:DIP-16_W7.62mm_Socket_LongPads
Connections:
- net +5V: now also J12.1 (Pin_1)
- net GND: now also J12.7 (Pin_7)
- net coarse2_a: now also J11.1 (Pin_1)
- net coarse3_a: now also J11.2 (Pin_2)
- net cvmod_a: now also J11.6 (Pin_6)
- net fine2_a: now also J11.3 (Pin_3)
- net fine3_a: now also J11.4 (Pin_4)
- net linfm_a: now also J11.5 (Pin_5)
- net pulse_a: now also J12.4 (Pin_4)
- net pwm_a: now also J12.2 (Pin_2)
- net saw_a: now also J12.5 (Pin_5)
- net sync_a: now also J12.3 (Pin_3)
- net tri_a: now also J12.6 (Pin_6)
- net voct_a: now also J11.7 (Pin_7)
