File: Dual_VCA/Kicad Project/Dual_VCA/Dual_VCA.kicad_sch (KiCad schematic)
At the start: 63 parts, among them J12 Conn_1A, J13 Conn_1B, J3 AUDIO_IN, J3 AUDIO_OUT, J3 CV_IN, J7 PWR, J8 Conn_2A, J9 Conn_2B, Q1 2N3904, Q2 2N3904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

Commit message: Recent updates for eurorack pcbs
Parts:
- removed J13: Conn_1B, Connector_PinHeader_2.54mm:PinHeader_1x04_P2.54mm_Vertical, symbol Connector:Conn_01x04_Pin
- removed J9: Conn_2B, Connector_PinHeader_2.54mm:PinHeader_1x04_P2.54mm_Vertical, symbol Connector:Conn_01x04_Pin
- added J10: Conn_1B, Connector_PinSocket_2.54mm:PinSocket_1x04_P2.54mm_Vertical, symbol Connector:Conn_01x04_Socket
- added J9: Conn_2B, Connector_PinSocket_2.54mm:PinSocket_1x04_P2.54mm_Vertical, symbol Connector:Conn_01x04_Socket
Connections:
- net GND: now also J10.1 (Pin_1)
- net cv1_a: now also J12.2 (Pin_2); no longer J12.4 (Pin_4)
- net cv1_b: now also J10.2 (Pin_2)
- net cv2_a: now also J8.2 (Pin_2); no longer J8.4 (Pin_4)
- net cv2_b: now also J9.2 (Pin_2)
- net in1_a: now also J12.4 (Pin_4); no longer J12.3 (Pin_3)
- net in1_b: now also J10.4 (Pin_4)
- net in2_b: now also J9.3 (Pin_3)
- net out1_a: now also J12.3 (Pin_3); no longer J12.2 (Pin_2)
- net out1_b: now also J10.3 (Pin_3)
- net out2_a: now also J8.4 (Pin_4); no longer J8.2 (Pin_2)
- net out2_b: now also J9.4 (Pin_4)
Changed lines of the file:
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@@
     (stroke (width 0) (type default))
   )
-  (wire (pts (xy 237.49 82.55) (xy 246.38 82.55))
-    (stroke (width 0) (type default))
-  )
   (wire (pts (xy 163.83 27.94) (xy 170.18 27.94))
     (stroke (width 0) (type default))
@@
     (stroke (width 0) (type default))
   )
+  (wire (pts (xy 237.49 82.55) (xy 246.38 82.55))
+    (stroke (width 0) (type default))
+  )
   (polyline (pts (xy 39.37 158.75) (xy 50.8 158.75))
     (stroke (width 0) (type default))
@@
     (stroke (width 0) (type default))
   )
-  (wire (pts (xy 246.38 82.55) (xy 246.38 83.82))
-    (stroke (width 0) (type default))
-  )
   (wire (pts (xy 81.28 149.86) (xy 81.28 161.29))
     (stroke (width 0) (type default))
@@
     (stroke (width 0) (type default))
   )
-  (wire (pts (xy 217.17 83.82) (xy 217.17 82.55))
-    (stroke (width 0) (type default))
-  )
   (wire (pts (xy 119.38 81.28) (xy 119.38 83.82))
     (stroke (width 0) (type default))
@@
     (stroke (width 0) (type default))
   )
+  (wire (pts (xy 217.17 82.55) (xy 226.06 82.55))
+    (stroke (width 0) (type default))
+  )
   (wire (pts (xy 81.28 161.29) (xy 83.82 161.29))
     (stroke (width 0) (type default))
@@
     (stroke (width 0) (type default))
   )
-  (wire (pts (xy 217.17 82.55) (xy 226.06 82.55))
-    (stroke (width 0) (type default))
-  )
   (wire (pts (xy 115.57 110.49) (xy 106.68 110.49))
     (stroke (width 0) (type default))
@@
     (stroke (width 0) (type default))
   )
+  (wire (pts (xy 217.17 85.09) (xy 217.17 82.55))
+    (stroke (width 0) (type default))
+  )
   (wire (pts (xy 229.87 105.41) (xy 232.41 105.41))
     (stroke (width 0) (type default))
@@
     (stroke (width 0) (type default))
   )
+  (wire (pts (xy 246.38 82.55) (xy 246.38 85.09))
+    (stroke (width 0) (type default))
+  )
   (wire (pts (xy 74.93 66.04) (xy 81.28 66.04))
     (stroke (width 0) (type default))
@@
     (effects (font (size 1.27 1.27)) (justify right bottom))
   )
-  (label "out1_a" (at 226.06 85.09 180) (fields_autoplaced)
+  (label "out1_a" (at 226.06 87.63 180) (fields_autoplaced)
     (effects (font (size 1.27 1.27)) (justify right bottom))
   )
@@
     (effects (font (size 1.27 1.27)) (justify left bottom))
   )
-  (label "cv1_a" (at 226.06 90.17 180) (fields_autoplaced)
+  (label "cv1_a" (at 226.06 85.09 180) (fields_autoplaced)
     (effects (font (size 1.27 1.27)) (justify right bottom))
   )
-  (label "out2_b" (at 266.7 85.09 0) (fields_autoplaced)
+  (label "out2_b" (at 266.7 90.17 0) (fields_autoplaced)
     (effects (font (size 1.27 1.27)) (justify left bottom))
   )
@@
     (effects (font (size 1.27 1.27)) (justify right bottom))
   )
-  (label "out2_a" (at 255.27 85.09 180) (fields_autoplaced)
+  (label "out2_a" (at 255.27 90.17 180) (fields_autoplaced)
     (effects (font (size 1.27 1.27)) (justify right bottom))
   )
@@
     (effects (font (size 1.27 1.27)) (justify left bottom))
   )
-  (label "in1_b" (at 237.49 87.63 0) (fields_autoplaced)
+  (label "in1_b" (at 237.49 90.17 0) (fields_autoplaced)
     (effects (font (size 1.27 1.27)) (justify left bottom))
   )
-  (label "cv2_b" (at 266.7 90.17 0) (fields_autoplaced)
+  (label "cv2_b" (at 266.7 85.09 0) (fields_autoplaced)
     (effects (font (size 1.27 1.27)) (justify left bottom))
   )
-  (label "cv2_a" (at 255.27 90.17 180) (fields_autoplaced)
+  (label "cv2_a" (at 255.27 85.09 180) (fields_autoplaced)
     (effects (font (size 1.27 1.27)) (justify right bottom))
   )
-  (label "cv1_b" (at 237.49 90.17 0) (fields_autoplaced)
+  (label "cv1_b" (at 237.49 85.09 0) (fields_autoplaced)
     (effects (font (size 1.27 1.27)) (justify left bottom))
   )
-  (label "out1_b" (at 237.49 85.09 0) (fields_autoplaced)
+  (label "out1_b" (at 237.49 87.63 0) (fields_autoplaced)
     (effects (font (size 1.27 1.27)) (justify left bottom))
   )
@@
     (effects (font (size 1.27 1.27)) (justify left bottom))
   )
-  (label "in1_a" (at 226.06 87.63 180) (fields_autoplaced)
+  (label "in1_a" (at 226.06 90.17 180) (fields_autoplaced)
     (effects (font (size 1.27 1.27)) (justify right bottom))
   )
@@
     )
   )
-  (symbol (lib_id "Connector:Conn_01x04_Pin") (at 232.41 85.09 0) (unit 1)
+  (symbol (lib_id "Connector:Conn_01x04_Socket") (at 261.62 85.09 0) (mirror y) (unit 1)
     (in_bom yes) (on_board yes) (dnp no)
-    (property "Reference" "J13" (at 234.95 78.74 0)
-      (effects (font (size 1.27 1.27)))
+    (property "Reference" "J9" (at 266.7 78.74 0)
+      (effects (font (size 1.27 1.27)) (justify left))
     )
-    (property "Value" "Conn_1B" (at 236.22 92.71 0)
-      (effects (font (size 1.27 1.27)))
+    (property "Value" "Conn_2B" (at 269.24 92.71 0)
+      (effects (font (size 1.27 1.27)) (justify left))
     )
-    (property "Footprint" "Connector_PinHeader_2.54mm:PinHeader_1x04_P2.54mm_Vertical" (at 232.41 85.09 0)
+    (property "Footprint" "Connector_PinSocket_2.54mm:PinSocket_1x04_P2.54mm_Vertical" (at 261.62 85.09 0)
       (effects (font (size 1.27 1.27)) hide)
     )
-    (property "Datasheet" "~" (at 232.41 85.09 0)
+    (property "Datasheet" "~" (at 261.62 85.09 0)
       (effects (font (size 1.27 1.27)) hide)
     )
@@
       (project "Dual_VCA"
         (path "/dcd60e2f-b4a3-409c-96a4-617c65996516"
-          (reference "J13") (unit 1)
+          (reference "J9") (unit 1)
         )
       )
@@
     )
   )
-  (symbol (lib_id "power:GND") (at 246.38 83.82 0) (unit 1)
+  (symbol (lib_id "power:GND") (at 246.38 85.09 0) (mirror y) (unit 1)
     (in_bom yes) (on_board yes) (dnp no) (fields_autoplaced)
-    (property "Reference" "#PWR047" (at 246.38 90.17 0)
+    (property "Reference" "#PWR047" (at 246.38 91.44 0)
       (effects (font (size 1.27 1.27)) hide)
     )
-    (property "Value" "GND" (at 246.38 88.9 0)
+    (property "Value" "GND" (at 246.38 90.17 0)
       (effects (font (size 1.27 1.27)) hide)
     )
-    (property "Footprint" "" (at 246.38 83.82 0)
+    (property "Footprint" "" (at 246.38 85.09 0)
       (effects (font (size 1.27 1.27)) hide)
     )
-    (property "Datasheet" "" (at 246.38 83.82 0)
+    (property "Datasheet" "" (at 246.38 85.09 0)
       (effects (font (size 1.27 1.27)) hide)
     )
@@
     )
   )
-  (symbol (lib_id "power:GND") (at 217.17 83.82 0) (unit 1)
+  (symbol (lib_id "power:GND") (at 217.17 85.09 0) (mirror y) (unit 1)
     (in_bom yes) (on_board yes) (dnp no) (fields_autoplaced)
-    (property "Reference" "#PWR046" (at 217.17 90.17 0)
+    (property "Reference" "#PWR046" (at 217.17 91.44 0)
       (effects (font (size 1.27 1.27)) hide)
     )
-    (property "Value" "GND" (at 217.17 88.9 0)
+    (property "Value" "GND" (at 217.17 90.17 0)
       (effects (font (size 1.27 1.27)) hide)
     )
-    (property "Footprint" "" (at 217.17 83.82 0)
+    (property "Footprint" "" (at 217.17 85.09 0)
       (effects (font (size 1.27 1.27)) hide)
     )
-    (property "Datasheet" "" (at 217.17 83.82 0)
+    (property "Datasheet" "" (at 217.17 85.09 0)
       (effects (font (size 1.27 1.27)) hide)
     )
@@
     )
   )
+  (symbol (lib_id "Connector:Conn_01x04_Socket") (at 232.41 85.09 0) (mirror y) (unit 1)
+    (in_bom yes) (on_board yes) (dnp no)
+    (property "Reference" "J10" (at 237.49 78.74 0)
+      (effects (font (size 1.27 1.27)) (justify left))
+    )
+    (property "Value" "Conn_1B" (at 240.03 92.71 0)
+      (effects (font (size 1.27 1.27)) (justify left))
+    )
+    (property "Footprint" "Connector_PinSocket_2.54mm:PinSocket_1x04_P2.54mm_Vertical" (at 232.41 85.09 0)
+      (effects (font (size 1.27 1.27)) hide)
+    )
+    (property "Datasheet" "~" (at 232.41 85.09 0)
+      (effects (font (size 1.27 1.27)) hide)
+    )
+    (pin "1")
+    (pin "2")
+    (pin "3")
+    (pin "4")
+    (instances
+      (project "Dual_VCA"
+        (path "/dcd60e2f-b4a3-409c-96a4-617c65996516"
+          (reference "J10") (unit 1)
+        )
+      )
+    )
+  )
   (symbol (lib_id "Device:R") (at 54.61 74.93 270) (mirror x) (unit 1)
     (in_bom yes) (on_board yes) (dnp no)
@@
         )
       )
-    )
-  )
-  (symbol (lib_id "Connector:Conn_01x04_Pin") (at 261.62 85.09 0) (unit 1)
-    (in_bom yes) (on_board yes) (dnp no)
-    (property "Reference" "J9" (at 264.16 78.74 0)
-      (effects (font (size 1.27 1.27)))
-    )
-    (property "Value" "Conn_2B" (at 265.43 92.71 0)
-      (effects (font (size 1.27 1.27)))
-    )
-    (property "Footprint" "Connector_PinHeader_2.54mm:PinHeader_1x04_P2.54mm_Vertical" (at 261.62 85.09 0)
-      (effects (font (size 1.27 1.27)) hide)
-    )
-    (property "Datasheet" "~" (at 261.62 85.09 0)
-      (effects (font (size 1.27 1.27)) hide)
-    )
-    (pin "1")
-    (pin "2")
-    (pin "3")
-    (pin "4")
-    (instances
-      (project "Dual_VCA"
-        (path "/dcd60e2f-b4a3-409c-96a4-617c65996516"
-          (reference "J9") (unit 1)
-        )
-      )
