File: 555_ADSR/Kicad_Project/555_ADSR/555_ADSR.kicad_sch (KiCad schematic)
At the start: 45 parts, among them J4 IN, J4 OUT1, J4 OUT2, J5 Conn1_a, J6 Conn1_b, J7 Conn1_a, J7 PWR, J8 Conn1_b, Q1 BC847, Q2 BC847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

Commit message: Updating project files
Connections:
- net GND: now also J7.3 (Pin_3), J7.5 (Pin_5), J7.7 (Pin_7)
Changed lines of the file:
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@@
+    )
+  )
+  (symbol (lib_id "power:GND") (at 130.81 251.46 0) (mirror y) (unit 1)
+    (in_bom yes) (on_board yes) (dnp no)
+    (property "Reference" "#PWR037" (at 130.81 257.81 0)
+      (effects (font (size 1.27 1.27)) hide)
+    )
+    (property "Value" "GND" (at 130.81 256.54 0)
+      (effects (font (size 1.27 1.27)))
+    )
+    (property "Footprint" "" (at 130.81 251.46 0)
+      (effects (font (size 1.27 1.27)) hide)
+    )
+    (property "Datasheet" "" (at 130.81 251.46 0)
+      (effects (font (size 1.27 1.27)) hide)
+    )
+    (pin "1")
+    (instances
+      (project "3340_VCO"
+        (path "/4db98d30-3bd7-4b4d-89f4-e727fe5b2269"
+          (reference "#PWR037") (unit 1)
+        )
+      )
+      (project "555_ADSR"
+        (path "/99a6a6a6-0bd7-49b0-8c76-b750d640b8ad"
+          (reference "#PWR035") (unit 1)
+        )
+      )
+      (project "CEM3340_VCO"
+        (path "/eb39d4cc-e98a-4977-a50e-25b815ed0a29"
+          (reference "#PWR0147") (unit 1)
+        )
+      )
     )
   )
